File: sunrise-board/sunrise-board.kicad_pcb (KiCad board)
At the start: 2 copper layers, 25.4 x 95.2 mm, 32 parts, among them J1 Barrel Jack 12V, J2 Header, J3 FTDI Basic, J4 Header, J5 LED_STRIP_VGRB, J6 I2C, Q1 IRLZ34N, Q2 IRLZ34N, Q3 IRLZ34N, SW1 Reset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

Commit message: fill and silk screen done
Parts:
- moved C6 0.59 mm to (132.6, 54.4)
- moved C3 0.51 mm to (132.6, 57.7)
- moved C4 0.51 mm to (145.3, 111.8)
- moved C5 0.51 mm to (145.3, 104.4)
- moved Y2 0.25 mm to (131.3, 113.0)
- moved R6 0.25 mm to (131.6, 125.2)
Routing:
- net D5: track 16.4 -> 13.7 mm
- net D7: track 11.2 -> 12.4 mm
- net VCC: track 182.5 -> 183.5 mm
- net D8: track 12.1 -> 11.4 mm
- net RESET: track 84.0 -> 83.4 mm
- added copper zone on B.Cu, net GND
- added copper zone on F.Cu, net GND
Other:
- board text added: "A0 A1"
- board text added: "A2 A3"
- board text added: "D12 SCK"
- board text added: "D2 D3"
- board text added: "D4 D5"
- board text added: "D6"
- board text added: "D7"
- board text added: "D8 D9"
- board text added: "D9 D6 D3 RAW"
- board text added: "FTDI"
- board text added: "GND"
- board text added: "GND RAW"
- board text added: "MISO MOSI"
- board text added: "RST GND"
- board text added: "SCK/D13"
- board text added: "SCL SDA"
- board text added: "SS D11"
- board text added: "Sunrise Alarm"
- board text added: "TXO RXI"
- board text added: "Tobin Yehle"
- board text added: "VCC RST"
- board text added: "v1"

Commit message: updates to silk screen
Other:
- board text added: "A4"
- board text added: "A5"
- board text added: "D2 ~D3~"
- board text added: "D3' RAW"
- board text added: "D8 ~D9~"
- board text added: "D9' D6'"
- board text added: "RAW"
- board text added: "VCC ~RST~"
- board text added: "~6~ 7"
- board text added: "~D6~"
- board text added: "~RST~ GND"
- board text removed: "D2 D3"
- board text removed: "D6"
- board text removed: "D7"
- board text removed: "D8 D9"
- board text removed: "D9 D6 D3 RAW"
- board text removed: "RST GND"
- board text removed: "VCC RST"
