File: hardware/sunrise-board.kicad_pcb (KiCad board)
At the start: 2 copper layers, 25.4 x 95.2 mm, 32 parts, among them J1 Barrel Jack 12V, J2 Header, J3 FTDI Basic, J4 Header, J5 LED_STRIP_VGRB, J6 I2C, Q1 IRLZ34N, Q2 IRLZ34N, Q3 IRLZ34N, SW1 Reset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

Commit message: fix crystal value
Parts:
- Y1: value 32.768Hz -> 32.768kHz
Changed lines of the file:
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@@
       (effects (font (size 1 1) (thickness 0.15)))
     )
-    (fp_text value 32.768Hz (at -1.016 5.334 270) (layer F.Fab)
+    (fp_text value 32.768kHz (at -1.016 5.334 270) (layer F.Fab)
       (effects (font (size 1 1) (thickness 0.15)))
     )
